File: Logic Gate/Logic Gate.kicad_sch (KiCad schematic)
At the start: 73 parts, among them J1 Barrel_Jack_MountingPin, Q1 PN2222A, Q10 PN2222A, Q11 PN2222A, Q12 PN2222A, Q13 PN2222A, Q14 PN2222A, Q15 PN2222A, Q16 PN2222A, Q17 PN2222A, Q18 PN2222A, Q2 PN2222A, Q3 PN2222A, Q4 PN2222A, Q5 PN2222A, Q6 PN2222A, Q7 PN2222A, Q8 PN2222A, Q9 PN2222A, SW1 SW_6x6x5, SW10 SW_6x6x5, SW11 SW_6x6x5, SW12 SW_6x6x5, SW13 SW_6x6x5, SW2 SW_6x6x5, SW3 SW_6x6x5, SW4 SW_6x6x5, SW5 SW_6x6x5, SW6 SW_6x6x5, SW7 SW_6x6x5, SW8 SW_6x6x5, SW9 SW_6x6x5, U1 L7805

Commit message: Traces revision
Parts:
- added J2: Conn_01x02_Socket, Connector_PinSocket_2.54mm:PinSocket_1x02_P2.54mm_Vertical, symbol Connector:Conn_01x02_Socket
Connections:
- net +5V: now also SW1.2, SW10.2, SW11.2, SW12.2, SW13.2, SW2.2, SW3.2, SW4.2, SW5.2, SW6.2, SW7.2, SW8.2, SW9.2, J2.1 (Pin_1); no longer SW1., SW10., SW11., SW12., SW13., SW2., SW3., SW4., SW5., SW6., SW7., SW8., SW9.
- net GND: now also J2.2 (Pin_2)
- net at R8.1: now also SW5.1; no longer SW5.
- net at R13.1: now also SW8.1; no longer SW8.
- net at R14.1: now also SW9.1; no longer SW9.
- net at R22.1, R23.1: now also SW13.1; no longer SW13.
- net at R2.1: now also SW2.1; no longer SW2.
- net at R10.1: now also SW6.1; no longer SW6.
- net at R16.1, R17.1, R19.1: now also SW10.1, SW11.1; no longer SW10., SW11.
- net at R21.1, R24.1: now also SW12.1; no longer SW12.
- net at R1.1: now also SW1.1; no longer SW1.
- net at R5.1: now also SW3.1; no longer SW3.
- net at R11.1: now also SW7.1; no longer SW7.
- net at R6.1: now also SW4.1; no longer SW4.
Other:
- note added: "ALTERNATIVE POWER"
- note added: "Optional Mounting Hole"
- moved on the sheet: C1, C2, D1, D2, D3, D4, D5, D6, D7, H1, H2, H3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

Commit message: minimum size
Parts:
- removed H1, H2, H3, H4: MountingHole, MountingHole:MountingHole_3.2mm_M3, symbol Mechanical:MountingHole
- removed R27: 330, Resistor_THT:R_Axial_DIN0309_L9.0mm_D3.2mm_P12.70mm_Horizontal, symbol Device:R_Small_US
- added D8: 1N4001, Diode_THT:D_DO-41_SOD81_P10.16mm_Horizontal, symbol Diode:1N4001
- R15: value 1k -> 330
Connections:
- net +5V: now also R26.1, D8.1 (K); no longer J2.1 (Pin_1)
- net at Q14.3 (C), Q16.3 (C), Q17.3 (C)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: no longer R26.1
- net at D6.2 (A), Q13.1 (E): now also Q12.1 (E)
- net at Q10.3 (C), R15.1: now also Q12.3 (C), Q13.3 (C); no longer R18.1
- net at R17.1, R19.1, SW11.1: no longer R16.1, SW10.1
- new net: D8.2 (A), J2.1 (Pin_1)
- new net: R16.1, R18.1, SW10.1
Other:
- note removed: "Optional Mounting Hole"
- moved on the sheet: D6, D7, Q12, R18, R26

Commit message: Backup
Parts:
- Q1, Q10, Q11, Q12, Q13, Q14, Q15, Q16, Q17, Q18, Q2, Q3, Q4, Q5, Q6, Q7, Q8, Q9: value PN2222A -> BC547
Other:
- moved on the sheet: C1, C2, D8, J1, J2, U1
